Commit message: Update proximity_sensor.urdf.xacro
Changed min range to 1 cm

File: thymio_description/urdf/proximity_sensor.urdf.xacro (robot description, xacro)
@@ -1,5 +1,5 @@
 <?xml version="1.0"?>
 <robot xmlns:xacro="http://playerstage.sourceforge.net/gazebo/xmlschema/#xacro">
-  <xacro:macro name="proximity_sensor" params="group name xyz rpy update_rate:=10 range_min:=0.00 range_max:=0.12 resolution:=0.005 fov:=0.3">
+  <xacro:macro name="proximity_sensor" params="group name xyz rpy update_rate:=10 range_min:=0.01 range_max:=0.12 resolution:=0.005 fov:=0.3">
     <link name="${group}_${name}_link"/>
     <joint name="${group}_${name}_joint" type="fixed">
