Commit message: Moved meshes to meters instead of inches, so that rviz is no more confused

File: thymio_description/urdf/wheel.urdf.xacro (robot description, xacro)
@@ -17,5 +17,5 @@
         <origin xyz="0 0 0" rpy="${pi/2 if name == 'left' else -pi/2} 0 0"/>
         <geometry>
-          <mesh filename="package://thymio_description/meshes/wheel.dae"/>
+          <mesh filename="package://thymio_description/meshes/wheel_inches.dae"/>
         </geometry>
       </visual>

Commit message: Moved meshes to meters instead of inches, so that rviz is no more confused

File: thymio_description/urdf/wheel.urdf.xacro (robot description, xacro)
@@ -17,5 +17,5 @@
         <origin xyz="0 0 0" rpy="${pi/2 if name == 'left' else -pi/2} 0 0"/>
         <geometry>
-          <mesh filename="package://thymio_description/meshes/wheel_inches.dae"/>
+          <mesh filename="package://thymio_description/meshes/wheel.dae"/>
         </geometry>
       </visual>
