Commit message: Completed description

File: thymio_description/urdf/base.urdf.xacro (robot description, xacro)
@@ -12,7 +12,7 @@
   <xacro:property name="wheel_torque" value="0.005"/>
   <!-- Body mass is 80% of total mass -->
-  <xacro:property name="body_mass" value="${mass * 0.80}"/>
+  <xacro:property name="body_mass" value="0.2"/>
   <!-- Each wheel is 10% of total mass -->
-  <xacro:property name="wheel_mass" value="${mass * 0.10}"/>
+  <xacro:property name="wheel_mass" value="0.024"/>
   <!-- <xacro:property name="base_radius" value="0.105"/>
   <xacro:property name="base_height" value="0.045"/> -->
@@ -20,7 +20,7 @@
     <link name="base_link">
       <inertial>
-        <origin xyz="0.025 0 0.009"/>
+        <origin xyz="0.0243 0 0.0315"/>
         <mass value="${body_mass}"/>
-        <inertia ixx="${0.0012141 * body_mass}" ixy="0" ixz="0" iyy="${0.0011771 * body_mass}" iyz="0" izz="${0.00205365 * body_mass}"/>
+        <inertia ixx="${0.002199 * body_mass}" ixy="0" ixz="-0.000760" iyy="${0.002639 * body_mass}" iyz="0" izz="${0.002526 * body_mass}"/>
       </inertial>
       <collision>
@@ -59,4 +59,10 @@
     <xacro:proximity_sensor group="ground" name="left" xyz="0.07157 0.01155 0.0009" rpy="0 1.5708 0.24311"/>
     <xacro:proximity_sensor group="ground" name="right" xyz="0.07157 -0.01155 0.0009" rpy="0 1.5708 -0.24311"/>
+    <link name="laser_link"/>
+    <joint name="base_laser_joint" type="fixed">
+      <parent link="base_link"/>
+      <child link="laser_link"/>
+      <origin xyz="0 0 0.035"/>
+    </joint>
     <xacro:imu/>
 <!-- see https://github.com/ros-simulation/gazebo_ros_pkgs/blob/kinetic-devel/gazebo_plugins/src/gazebo_ros_diff_drive.cpp -->

File: thymio_description/urdf/wheel.urdf.xacro (robot description, xacro)
@@ -1,5 +1,5 @@
 <?xml version="1.0"?>
 <robot xmlns:xacro="http://playerstage.sourceforge.net/gazebo/xmlschema/#xacro">
-  <xacro:macro name="wheel" params="name position mass:=0.02 mu:=100 radius:=0.022 width=0.015">
+  <xacro:macro name="wheel" params="name position mass:=0.024 mu:=100 radius:=0.022 width=0.015 max_speed=7.757">
     <link name="${name}_wheel_link">
       <inertial>
@@ -26,4 +26,5 @@
       <axis xyz="0 1 0"/>
       <origin xyz="0 ${position} ${radius}"/>
+      <limit velocity="${max_speed}" effort="0"/>
     </joint>
     <gazebo reference="${name}_wheel_link">

Commit message: Completed description

File: thymio_description/urdf/base.urdf.xacro (robot description, xacro)
@@ -15,6 +15,5 @@
   <!-- Each wheel is 10% of total mass -->
   <xacro:property name="wheel_mass" value="0.024"/>
-  <!-- <xacro:property name="base_radius" value="0.105"/>
-  <xacro:property name="base_height" value="0.045"/> -->
+  <!-- <xacro:property name="base_radius" value="0.105"/> <xacro:property name="base_height" value="0.045"/> -->
   <xacro:macro name="thymio">
     <link name="base_link">
@@ -22,5 +21,5 @@
         <origin xyz="0.0243 0 0.0315"/>
         <mass value="${body_mass}"/>
-        <inertia ixx="${0.002199 * body_mass}" ixy="0" ixz="-0.000760" iyy="${0.002639 * body_mass}" iyz="0" izz="${0.002526 * body_mass}"/>
+        <inertia ixx="${0.002199 * body_mass}" ixy="0" ixz="${-0.000760 * body_mass}" iyy="${0.002639 * body_mass}" iyz="0" izz="${0.002526 * body_mass}"/>
       </inertial>
       <collision>
@@ -39,12 +38,12 @@
         <origin xyz="0.0 0 0.0" rpy="0 0 0"/>
         <geometry>
-          <mesh filename="package://thymio_description/meshes/base_essential_3.dae"/>
+          <mesh filename="package://thymio_description/meshes/base_simple.dae"/>
         </geometry>
       </visual>
     </link>
     <gazebo reference="base_link">
-      <selfCollide>true</selfCollide>
-      <mu1>0.0</mu1>
-      <mu2>0.0</mu2>5
+      <selfCollide>false</selfCollide>
+      <mu1>0.1</mu1>
+      <mu2>0.1</mu2>
     </gazebo>
     <xacro:wheel name="left" position="${wheel_axis * 0.5}" radius="${wheel_radius}" mass="${wheel_mass}" mu="$(arg left_wheel_mu)"/>
@@ -57,6 +56,6 @@
     <xacro:proximity_sensor group="proximity" name="rear_left" xyz="-0.03 0.0305 0.035" rpy="0 0 3.14159"/>
     <xacro:proximity_sensor group="proximity" name="rear_right" xyz="-0.03 -0.0305 0.035" rpy="0 0 3.14159"/>
-    <xacro:proximity_sensor group="ground" name="left" xyz="0.07157 0.01155 0.0009" rpy="0 1.5708 0.24311"/>
-    <xacro:proximity_sensor group="ground" name="right" xyz="0.07157 -0.01155 0.0009" rpy="0 1.5708 -0.24311"/>
+    <xacro:proximity_sensor group="ground" range_max="0.03" name="left" xyz="0.07157 0.01155 0.0009" rpy="0 1.5708 0.24311"/>
+    <xacro:proximity_sensor group="ground" range_max="0.03" name="right" xyz="0.07157 -0.01155 0.0009" rpy="0 1.5708 -0.24311"/>
     <link name="laser_link"/>
     <joint name="base_laser_joint" type="fixed">
@@ -66,5 +65,5 @@
     </joint>
     <xacro:imu/>
-<!-- see https://github.com/ros-simulation/gazebo_ros_pkgs/blob/kinetic-devel/gazebo_plugins/src/gazebo_ros_diff_drive.cpp -->
+    <!-- see https://github.com/ros-simulation/gazebo_ros_pkgs/blob/kinetic-devel/gazebo_plugins/src/gazebo_ros_diff_drive.cpp -->
     <gazebo>
       <plugin name="differential_drive_controller" filename="libgazebo_ros_diff_drive.so">
@@ -74,6 +73,6 @@
         <alwaysOn>true</alwaysOn>
         <updateRate>100</updateRate>
-        <leftJoint>right_wheel_joint</leftJoint>
-        <rightJoint>left_wheel_joint</rightJoint>
+        <leftJoint>left_wheel_joint</leftJoint>
+        <rightJoint>right_wheel_joint</rightJoint>
         <wheelSeparation>${wheel_axis}</wheelSeparation>
         <wheelDiameter>${2 * wheel_radius}</wheelDiameter>
@@ -89,12 +88,5 @@
       </plugin>
     </gazebo>
-    <!-- <gazebo>
-  <plugin name="ground_truth" filename="libgazebo_ros_p3d.so">
-    <frameName>world</frameName>
-    <bodyName>base_link</bodyName>
-    <topicName>ground_truth</topicName>
-    <updateRate>30.0</updateRate>
-  </plugin>
-  </gazebo> -->
+    <!-- <gazebo> <plugin name="ground_truth" filename="libgazebo_ros_p3d.so"> <frameName>world</frameName> <bodyName>base_link</bodyName> <topicName>ground_truth</topicName> <updateRate>30.0</updateRate> </plugin> </gazebo> -->
   </xacro:macro>
 </robot>

Commit message: Added tf namespace to IMU

File: thymio_description/urdf/base.urdf.xacro (robot description, xacro)
@@ -6,13 +6,10 @@
   <xacro:arg name="left_wheel_mu" default="100.0"/>
   <xacro:arg name="right_wheel_mu" default="100.0"/>
-  <xacro:arg name="mass" default="0.200"/>
-  <xacro:property name="mass" value="$(arg mass)"/>
   <xacro:property name="wheel_axis" value="0.095"/>
   <xacro:property name="wheel_radius" value="0.022"/>
   <xacro:property name="wheel_torque" value="0.005"/>
-  <!-- Body mass is 80% of total mass -->
   <xacro:property name="body_mass" value="0.2"/>
-  <!-- Each wheel is 10% of total mass -->
   <xacro:property name="wheel_mass" value="0.024"/>
+  <xacro:arg name="name" default=""/>
   <!-- <xacro:property name="base_radius" value="0.105"/> <xacro:property name="base_height" value="0.045"/> -->
   <xacro:macro name="thymio">
@@ -64,5 +61,5 @@
       <origin xyz="0 0 0.035"/>
     </joint>
-    <xacro:imu/>
+    <xacro:imu ns="$(arg name)"/>
     <!-- see https://github.com/ros-simulation/gazebo_ros_pkgs/blob/kinetic-devel/gazebo_plugins/src/gazebo_ros_diff_drive.cpp -->
     <gazebo>

File: thymio_description/urdf/imu.urdf.xacro (robot description, xacro)
@@ -1,5 +1,5 @@
 <?xml version="1.0"?>
 <robot xmlns:xacro="http://playerstage.sourceforge.net/gazebo/xmlschema/#xacro">
-  <xacro:macro name="imu">
+  <xacro:macro name="imu" params="ns">
     <gazebo reference="base_link">
       <gravity>true</gravity>
@@ -16,5 +16,5 @@
           <xyzOffset>0 0 0</xyzOffset>
           <rpyOffset>0 0 0</rpyOffset>
-          <frameName>base_link</frameName>
+          <frameName>${ns}base_link</frameName>
         </plugin>
         <pose>0 0 0 0 0 0</pose>

Commit message: Adjusted axis length

File: thymio_description/urdf/base.urdf.xacro (robot description, xacro)
@@ -6,5 +6,5 @@
   <xacro:arg name="left_wheel_mu" default="100.0"/>
   <xacro:arg name="right_wheel_mu" default="100.0"/>
-  <xacro:property name="wheel_axis" value="0.095"/>
+  <xacro:property name="wheel_axis" value="0.0935"/>
   <xacro:property name="wheel_radius" value="0.022"/>
   <xacro:property name="wheel_torque" value="0.005"/>

Commit message: Exposed proximity params

File: thymio_description/urdf/base.urdf.xacro (robot description, xacro)
@@ -11,6 +11,7 @@
   <xacro:property name="body_mass" value="0.2"/>
   <xacro:property name="wheel_mass" value="0.024"/>
+  <xacro:arg name="proximity_max_range" default="0.12"/>
+  <xacro:arg name="proximity_resolution" default="0.005"/>
   <xacro:arg name="name" default=""/>
-  <!-- <xacro:property name="base_radius" value="0.105"/> <xacro:property name="base_height" value="0.045"/> -->
   <xacro:macro name="thymio">
     <link name="base_link">
@@ -46,11 +47,11 @@
     <xacro:wheel name="left" position="${wheel_axis * 0.5}" radius="${wheel_radius}" mass="${wheel_mass}" mu="$(arg left_wheel_mu)"/>
     <xacro:wheel name="right" position="${-wheel_axis * 0.5}" radius="${wheel_radius}" mass="${wheel_mass}" mu="$(arg right_wheel_mu)"/>
-    <xacro:proximity_sensor group="proximity" name="center" xyz="0.08 0 0.035" rpy="0 0 0"/>
-    <xacro:proximity_sensor group="proximity" name="center_left" xyz="0.0756 0.0261 0.035" rpy="0 0 0.33161"/>
-    <xacro:proximity_sensor group="proximity" name="center_right" xyz="0.0756 -0.0261 0.035" rpy="0 0 -0.33161"/>
-    <xacro:proximity_sensor group="proximity" name="left" xyz="0.063 0.0493 0.035" rpy="0 0 0.66323"/>
-    <xacro:proximity_sensor group="proximity" name="right" xyz="0.063 -0.0493 0.035" rpy="0 0 -0.66323"/>
-    <xacro:proximity_sensor group="proximity" name="rear_left" xyz="-0.03 0.0305 0.035" rpy="0 0 3.14159"/>
-    <xacro:proximity_sensor group="proximity" name="rear_right" xyz="-0.03 -0.0305 0.035" rpy="0 0 3.14159"/>
+    <xacro:proximity_sensor group="proximity" range_max="${arg proximity_max_range}" resolutio="${arg proximity_resolution}" name="center" xyz="0.08 0 0.035" rpy="0 0 0"/>
+    <xacro:proximity_sensor group="proximity" range_max="${arg proximity_max_range}" resolutio="${arg proximity_resolution}" name="center_left" xyz="0.0756 0.0261 0.035" rpy="0 0 0.33161"/>
+    <xacro:proximity_sensor group="proximity" range_max="${arg proximity_max_range}" resolutio="${arg proximity_resolution}" name="center_right" xyz="0.0756 -0.0261 0.035" rpy="0 0 -0.33161"/>
+    <xacro:proximity_sensor group="proximity" range_max="${arg proximity_max_range}" resolutio="${arg proximity_resolution}" name="left" xyz="0.063 0.0493 0.035" rpy="0 0 0.66323"/>
+    <xacro:proximity_sensor group="proximity" range_max="${arg proximity_max_range}" resolutio="${arg proximity_resolution}" name="right" xyz="0.063 -0.0493 0.035" rpy="0 0 -0.66323"/>
+    <xacro:proximity_sensor group="proximity" range_max="${arg proximity_max_range}" resolutio="${arg proximity_resolution}" name="rear_left" xyz="-0.03 0.0305 0.035" rpy="0 0 3.14159"/>
+    <xacro:proximity_sensor group="proximity" range_max="${arg proximity_max_range}" resolutio="${arg proximity_resolution}" name="rear_right" xyz="-0.03 -0.0305 0.035" rpy="0 0 3.14159"/>
     <xacro:proximity_sensor group="ground" range_max="0.03" name="left" xyz="0.07157 0.01155 0.0009" rpy="0 1.5708 0.24311"/>
     <xacro:proximity_sensor group="ground" range_max="0.03" name="right" xyz="0.07157 -0.01155 0.0009" rpy="0 1.5708 -0.24311"/>

Commit message: Added odom_max_rate. Added (gazebo) odom ground truth

File: thymio_description/urdf/base.urdf.xacro (robot description, xacro)
@@ -8,5 +8,5 @@
   <xacro:property name="wheel_axis" value="0.0935"/>
   <xacro:property name="wheel_radius" value="0.022"/>
-  <xacro:property name="wheel_torque" value="0.005"/>
+  <xacro:property name="wheel_torque" value="50"/>
   <xacro:property name="body_mass" value="0.2"/>
   <xacro:property name="wheel_mass" value="0.024"/>
@@ -15,4 +15,8 @@
   <xacro:arg name="proximity_fov" default="0.3"/>
   <xacro:arg name="name" default=""/>
+  <xacro:arg name="publish_ground_truth" default="false"/>
+  <xacro:arg name="ground_truth_frame_id" default="/world"/>
+  <xacro:arg name="ground_truth_update_rate" default="10.0"/>
+  <xacro:arg name="odom_max_rate" default="20.0"/>
   <xacro:macro name="thymio">
     <link name="base_link">
@@ -71,5 +75,5 @@
         <odometrySource>encoder</odometrySource>
         <alwaysOn>true</alwaysOn>
-        <updateRate>100</updateRate>
+        <updateRate>$(arg odom_max_rate)</updateRate>
         <leftJoint>left_wheel_joint</leftJoint>
         <rightJoint>right_wheel_joint</rightJoint>
@@ -87,5 +91,17 @@
       </plugin>
     </gazebo>
-    <!-- <gazebo> <plugin name="ground_truth" filename="libgazebo_ros_p3d.so"> <frameName>world</frameName> <bodyName>base_link</bodyName> <topicName>ground_truth</topicName> <updateRate>30.0</updateRate> </plugin> </gazebo> -->
+    <!-- NOTE: The current version of the gazebo p3d plugin has a bug:
+    the field child_frame_id is set to the name of the link (bodyName)
+    and not to the frame name (frameName). -->
+    <xacro:if value="$(arg publish_ground_truth)">
+      <gazebo>
+        <plugin name="ground_truth" filename="libgazebo_ros_p3d.so">
+          <frameName>$(arg ground_truth_frame_id)</frameName>
+          <bodyName>base_link</bodyName>
+          <topicName>ground_truth/odom</topicName>
+          <updateRate>$(arg ground_truth_update_rate)</updateRate>
+        </plugin>
+      </gazebo>
+     </xacro:if>
   </xacro:macro>
 </robot>

File: thymio_description/urdf/wheel.urdf.xacro (robot description, xacro)
@@ -27,4 +27,5 @@
       <origin xyz="0 ${position} ${radius}"/>
       <limit velocity="${max_speed}" effort="0"/>
+      <dynamics damping="0.1" friction="0.1"/>
     </joint>
     <gazebo reference="${name}_wheel_link">

Commit message: Added odom max rate

File: thymio_description/urdf/base.urdf.xacro (robot description, xacro)
@@ -8,5 +8,5 @@
   <xacro:property name="wheel_axis" value="0.0935"/>
   <xacro:property name="wheel_radius" value="0.022"/>
-  <xacro:property name="wheel_torque" value="50"/>
+  <xacro:property name="wheel_torque" value="0.1"/>
   <xacro:property name="body_mass" value="0.2"/>
   <xacro:property name="wheel_mass" value="0.024"/>

Commit message: Added kp

File: thymio_description/urdf/base.urdf.xacro (robot description, xacro)
@@ -4,10 +4,12 @@
   <xacro:include filename="$(find thymio_description)/urdf/proximity_sensor.urdf.xacro"/>
   <xacro:include filename="$(find thymio_description)/urdf/imu.urdf.xacro"/>
-  <xacro:arg name="left_wheel_mu" default="100.0"/>
-  <xacro:arg name="right_wheel_mu" default="100.0"/>
+  <xacro:arg name="left_wheel_mu" default="1.0"/>
+  <xacro:arg name="right_wheel_mu" default="1.0"/>
   <xacro:property name="wheel_axis" value="0.0935"/>
   <xacro:property name="wheel_radius" value="0.022"/>
   <xacro:property name="wheel_torque" value="0.1"/>
+  <xacro:property name="wheel_kp" value="10000"/>
   <xacro:property name="body_mass" value="0.2"/>
+  <xacro:property name="body_kp" value="17500"/>
   <xacro:property name="wheel_mass" value="0.024"/>
   <xacro:arg name="proximity_max_range" default="0.12"/>
@@ -22,5 +24,5 @@
     <link name="base_link">
       <inertial>
-        <origin xyz="0.0243 0 0.0315"/>
+        <origin xyz="0.0243 0 0.0205"/>
         <mass value="${body_mass}"/>
         <inertia ixx="${0.002199 * body_mass}" ixy="0" ixz="${-0.000760 * body_mass}" iyy="${0.002639 * body_mass}" iyz="0" izz="${0.002526 * body_mass}"/>
@@ -49,4 +51,6 @@
       <mu1>0.1</mu1>
       <mu2>0.1</mu2>
+      <kp>$(arg body_kp)</kp>
+      <kd>1</kd>
     </gazebo>
     <xacro:wheel name="left" position="${wheel_axis * 0.5}" radius="${wheel_radius}" mass="${wheel_mass}" mu="$(arg left_wheel_mu)"/>

File: thymio_description/urdf/wheel.urdf.xacro (robot description, xacro)
@@ -1,5 +1,5 @@
 <?xml version="1.0"?>
 <robot xmlns:xacro="http://playerstage.sourceforge.net/gazebo/xmlschema/#xacro">
-  <xacro:macro name="wheel" params="name position mass:=0.024 mu:=100 radius:=0.022 width=0.015 max_speed=7.757">
+  <xacro:macro name="wheel" params="name position mass:=0.024 mu:=100 radius:=0.022 width=0.015 max_speed=7.757 kp=10000">
     <link name="${name}_wheel_link">
       <inertial>
@@ -27,9 +27,11 @@
       <origin xyz="0 ${position} ${radius}"/>
       <limit velocity="${max_speed}" effort="0"/>
-      <dynamics damping="0.1" friction="0.1"/>
+      <!-- <dynamics damping="0.1" friction="0.1"/> -->
     </joint>
     <gazebo reference="${name}_wheel_link">
       <mu1>${mu}</mu1>
       <mu2>${mu / 2.0}</mu2>
+      <kp>${kp}</kp>
+      <kd>1</kd>
     </gazebo>
   </xacro:macro>

Commit message: Added kp

File: thymio_description/urdf/base.urdf.xacro (robot description, xacro)
@@ -9,7 +9,7 @@
   <xacro:property name="wheel_radius" value="0.022"/>
   <xacro:property name="wheel_torque" value="0.1"/>
-  <xacro:property name="wheel_kp" value="10000"/>
+  <xacro:arg name="wheel_kp" value="10000"/>
   <xacro:property name="body_mass" value="0.2"/>
-  <xacro:property name="body_kp" value="17500"/>
+  <xacro:arg name="body_kp" value="17500"/>
   <xacro:property name="wheel_mass" value="0.024"/>
   <xacro:arg name="proximity_max_range" default="0.12"/>
@@ -54,6 +54,6 @@
       <kd>1</kd>
     </gazebo>
-    <xacro:wheel name="left" position="${wheel_axis * 0.5}" radius="${wheel_radius}" mass="${wheel_mass}" mu="$(arg left_wheel_mu)"/>
-    <xacro:wheel name="right" position="${-wheel_axis * 0.5}" radius="${wheel_radius}" mass="${wheel_mass}" mu="$(arg right_wheel_mu)"/>
+    <xacro:wheel name="left" position="${wheel_axis * 0.5}" radius="${wheel_radius}" mass="${wheel_mass}" mu="$(arg left_wheel_mu)" kp="$(arg wheel_kp)"/>
+    <xacro:wheel name="right" position="${-wheel_axis * 0.5}" radius="${wheel_radius}" mass="${wheel_mass}" mu="$(arg right_wheel_mu)" kp="$(arg wheel_kp)"/>
     <xacro:proximity_sensor group="proximity" range_max="$(arg proximity_max_range)" resolution="$(arg proximity_resolution)" fov="$(arg proximity_fov)" name="center" xyz="0.08 0 0.035" rpy="0 0 0"/>
     <xacro:proximity_sensor group="proximity" range_max="$(arg proximity_max_range)" resolution="$(arg proximity_resolution)" fov="$(arg proximity_fov)" name="center_left" xyz="0.0756 0.0261 0.035" rpy="0 0 0.33161"/>

Commit message: Solved drifting issues (with kp), deformation issues (with narrower wheel) and wrong odometry angular speed (with axis = wheel dist + wheel width)

File: thymio_description/urdf/base.urdf.xacro (robot description, xacro)
@@ -7,4 +7,5 @@
   <xacro:arg name="right_wheel_mu" default="1.0"/>
   <xacro:property name="wheel_axis" value="0.0935"/>
+  <xacro:arg name="wheel_width" default="0.00015"/>
   <xacro:property name="wheel_radius" value="0.022"/>
   <xacro:property name="wheel_torque" value="0.1"/>
@@ -54,7 +55,7 @@
       <kd>1</kd>
     </gazebo>
-    <xacro:wheel name="left" position="${wheel_axis * 0.5}" radius="${wheel_radius}" mass="${wheel_mass}" mu="$(arg left_wheel_mu)" kp="$(arg wheel_kp)"/>
-    <xacro:wheel name="right" position="${-wheel_axis * 0.5}" radius="${wheel_radius}" mass="${wheel_mass}" mu="$(arg right_wheel_mu)" kp="$(arg wheel_kp)"/>
-    <xacro:proximity_sensor group="proximity" range_max="$(arg proximity_max_range)" resolution="$(arg proximity_resolution)" fov="$(arg proximity_fov)" name="center" xyz="0.08 0 0.035" rpy="0 0 0"/>
+    <xacro:wheel name="left" position="${wheel_axis * 0.5}" radius="${wheel_radius}" mass="${wheel_mass}" mu="$(arg left_wheel_mu)" kp="$(arg wheel_kp)" width="$(arg wheel_width)"/>
+    <xacro:wheel name="right" position="${-wheel_axis * 0.5}" radius="${wheel_radius}" mass="${wheel_mass}" mu="$(arg right_wheel_mu)" kp="$(arg wheel_kp)" width="$(arg wheel_width)"/>
+  <xacro:proximity_sensor group="proximity" range_max="$(arg proximity_max_range)" resolution="$(arg proximity_resolution)" fov="$(arg proximity_fov)" name="center" xyz="0.08 0 0.035" rpy="0 0 0"/>
     <xacro:proximity_sensor group="proximity" range_max="$(arg proximity_max_range)" resolution="$(arg proximity_resolution)" fov="$(arg proximity_fov)" name="center_left" xyz="0.0756 0.0261 0.035" rpy="0 0 0.33161"/>
     <xacro:proximity_sensor group="proximity" range_max="$(arg proximity_max_range)" resolution="$(arg proximity_resolution)" fov="$(arg proximity_fov)" name="center_right" xyz="0.0756 -0.0261 0.035" rpy="0 0 -0.33161"/>
@@ -82,5 +83,5 @@
         <leftJoint>left_wheel_joint</leftJoint>
         <rightJoint>right_wheel_joint</rightJoint>
-        <wheelSeparation>${wheel_axis}</wheelSeparation>
+        <wheelSeparation>${wheel_axis + wheel_width}</wheelSeparation>
         <wheelDiameter>${2 * wheel_radius}</wheelDiameter>
         <wheelTorque>${wheel_torque}</wheelTorque>

File: thymio_description/urdf/wheel.urdf.xacro (robot description, xacro)
@@ -26,5 +26,5 @@
       <axis xyz="0 1 0"/>
       <origin xyz="0 ${position} ${radius}"/>
-      <limit velocity="${max_speed}" effort="0"/>
+      <!-- <limit velocity="${max_speed}" effort="0"/> -->
       <!-- <dynamics damping="0.1" friction="0.1"/> -->
     </joint>

Commit message: Local change

File: thymio_description/urdf/base.urdf.xacro (robot description, xacro)
@@ -8,9 +8,10 @@
   <xacro:property name="wheel_axis" value="0.0935"/>
   <xacro:arg name="wheel_width" default="0.00015"/>
+  <xacro:property name="r_wheel_width" value="$(arg wheel_width)"/>
   <xacro:property name="wheel_radius" value="0.022"/>
   <xacro:property name="wheel_torque" value="0.1"/>
-  <xacro:arg name="wheel_kp" default="10000"/>
+  <xacro:arg name="wheel_kp" default="100000"/>
   <xacro:property name="body_mass" value="0.2"/>
-  <xacro:arg name="body_kp" default="17500"/>
+  <xacro:arg name="body_kp" default="175000"/>
   <xacro:property name="wheel_mass" value="0.024"/>
   <xacro:arg name="proximity_max_range" default="0.12"/>
@@ -83,5 +84,5 @@
         <leftJoint>left_wheel_joint</leftJoint>
         <rightJoint>right_wheel_joint</rightJoint>
-        <wheelSeparation>${wheel_axis + wheel_width}</wheelSeparation>
+        <wheelSeparation>${wheel_axis + 0 * r_wheel_width}</wheelSeparation>
         <wheelDiameter>${2 * wheel_radius}</wheelDiameter>
         <wheelTorque>${wheel_torque}</wheelTorque>
