Commit message: Updated to ROS1 Noetic

File: thymio_description/urdf/base.urdf.xacro (robot description, xacro)
@@ -24,5 +24,5 @@
   <xacro:arg name="odom_max_rate" default="20.0"/>
   <xacro:macro name="thymio">
-    <link name="base_link">
+    <link name="body_link">
       <inertial>
         <origin xyz="0.0243 0 0.0205"/>
@@ -49,4 +49,11 @@
       </visual>
     </link>
+    <link name="base_link">
+    </link>
+    <joint name="body_joint" type="fixed">
+      <parent link="base_link"/>
+      <child link="body_link"/>
+      <origin xyz="0 0 0"/>
+    </joint>
     <gazebo reference="base_link">
       <selfCollide>false</selfCollide>
@@ -58,5 +65,5 @@
     <xacro:wheel name="left" position="${wheel_axis * 0.5}" radius="${wheel_radius}" mass="${wheel_mass}" mu="$(arg left_wheel_mu)" kp="$(arg wheel_kp)" width="$(arg wheel_width)"/>
     <xacro:wheel name="right" position="${-wheel_axis * 0.5}" radius="${wheel_radius}" mass="${wheel_mass}" mu="$(arg right_wheel_mu)" kp="$(arg wheel_kp)" width="$(arg wheel_width)"/>
-  <xacro:proximity_sensor group="proximity" range_max="$(arg proximity_max_range)" resolution="$(arg proximity_resolution)" fov="$(arg proximity_fov)" name="center" xyz="0.08 0 0.035" rpy="0 0 0"/>
+    <xacro:proximity_sensor group="proximity" range_max="$(arg proximity_max_range)" resolution="$(arg proximity_resolution)" fov="$(arg proximity_fov)" name="center" xyz="0.08 0 0.035" rpy="0 0 0"/>
     <xacro:proximity_sensor group="proximity" range_max="$(arg proximity_max_range)" resolution="$(arg proximity_resolution)" fov="$(arg proximity_fov)" name="center_left" xyz="0.0756 0.0261 0.035" rpy="0 0 0.33161"/>
     <xacro:proximity_sensor group="proximity" range_max="$(arg proximity_max_range)" resolution="$(arg proximity_resolution)" fov="$(arg proximity_fov)" name="center_right" xyz="0.0756 -0.0261 0.035" rpy="0 0 -0.33161"/>
@@ -81,4 +88,5 @@
         <odometrySource>encoder</odometrySource>
         <alwaysOn>true</alwaysOn>
+        <publishOdomTF>false</publishOdomTF>
         <updateRate>$(arg odom_max_rate)</updateRate>
         <leftJoint>left_wheel_joint</leftJoint>

Commit message: Replaced deprecated implicit with explicit tf_prefix

File: thymio_description/urdf/base.urdf.xacro (robot description, xacro)
@@ -23,6 +23,13 @@
   <xacro:arg name="ground_truth_update_rate" default="10.0"/>
   <xacro:arg name="odom_max_rate" default="20.0"/>
+  <xacro:property name="_name" value="$(arg name)"/>
+  <xacro:if value="${_name != ''}">
+    <xacro:property name="tf_prefix" value="${_name}/"/>
+  </xacro:if>
+  <xacro:if value="${_name == ''}">
+    <xacro:property name="tf_prefix" value=""/>
+  </xacro:if>
   <xacro:macro name="thymio">
-    <link name="body_link">
+    <link name="${tf_prefix}body_link">
       <inertial>
         <origin xyz="0.0243 0 0.0205"/>
@@ -49,12 +56,12 @@
       </visual>
     </link>
-    <link name="base_link">
+    <link name="${tf_prefix}base_link">
     </link>
-    <joint name="body_joint" type="fixed">
-      <parent link="base_link"/>
-      <child link="body_link"/>
+    <joint name="${tf_prefix}body_joint" type="fixed">
+      <parent link="${tf_prefix}base_link"/>
+      <child link="${tf_prefix}body_link"/>
       <origin xyz="0 0 0"/>
     </joint>
-    <gazebo reference="base_link">
+    <gazebo reference="${tf_prefix}base_link">
       <selfCollide>false</selfCollide>
       <mu1>0.1</mu1>
@@ -63,22 +70,22 @@
       <kd>1</kd>
     </gazebo>
-    <xacro:wheel name="left" position="${wheel_axis * 0.5}" radius="${wheel_radius}" mass="${wheel_mass}" mu="$(arg left_wheel_mu)" kp="$(arg wheel_kp)" width="$(arg wheel_width)"/>
-    <xacro:wheel name="right" position="${-wheel_axis * 0.5}" radius="${wheel_radius}" mass="${wheel_mass}" mu="$(arg right_wheel_mu)" kp="$(arg wheel_kp)" width="$(arg wheel_width)"/>
-    <xacro:proximity_sensor group="proximity" range_max="$(arg proximity_max_range)" resolution="$(arg proximity_resolution)" fov="$(arg proximity_fov)" name="center" xyz="0.08 0 0.035" rpy="0 0 0"/>
-    <xacro:proximity_sensor group="proximity" range_max="$(arg proximity_max_range)" resolution="$(arg proximity_resolution)" fov="$(arg proximity_fov)" name="center_left" xyz="0.0756 0.0261 0.035" rpy="0 0 0.33161"/>
-    <xacro:proximity_sensor group="proximity" range_max="$(arg proximity_max_range)" resolution="$(arg proximity_resolution)" fov="$(arg proximity_fov)" name="center_right" xyz="0.0756 -0.0261 0.035" rpy="0 0 -0.33161"/>
-    <xacro:proximity_sensor group="proximity" range_max="$(arg proximity_max_range)" resolution="$(arg proximity_resolution)" fov="$(arg proximity_fov)" name="left" xyz="0.063 0.0493 0.035" rpy="0 0 0.66323"/>
-    <xacro:proximity_sensor group="proximity" range_max="$(arg proximity_max_range)" resolution="$(arg proximity_resolution)" fov="$(arg proximity_fov)" name="right" xyz="0.063 -0.0493 0.035" rpy="0 0 -0.66323"/>
-    <xacro:proximity_sensor group="proximity" range_max="$(arg proximity_max_range)" resolution="$(arg proximity_resolution)" fov="$(arg proximity_fov)" name="rear_left" xyz="-0.03 0.0305 0.035" rpy="0 0 3.14159"/>
-    <xacro:proximity_sensor group="proximity" range_max="$(arg proximity_max_range)" resolution="$(arg proximity_resolution)" fov="$(arg proximity_fov)" name="rear_right" xyz="-0.03 -0.0305 0.035" rpy="0 0 3.14159"/>
-    <xacro:proximity_sensor group="ground" range_max="0.03" name="left" xyz="0.07157 0.01155 0.0009" rpy="0 1.5708 0.24311"/>
-    <xacro:proximity_sensor group="ground" range_max="0.03" name="right" xyz="0.07157 -0.01155 0.0009" rpy="0 1.5708 -0.24311"/>
-    <link name="laser_link"/>
-    <joint name="base_laser_joint" type="fixed">
-      <parent link="base_link"/>
-      <child link="laser_link"/>
+    <xacro:wheel tf_prefix="${tf_prefix}" name="left" position="${wheel_axis * 0.5}" radius="${wheel_radius}" mass="${wheel_mass}" mu="$(arg left_wheel_mu)" kp="$(arg wheel_kp)" width="$(arg wheel_width)"/>
+    <xacro:wheel tf_prefix="${tf_prefix}" name="right" position="${-wheel_axis * 0.5}" radius="${wheel_radius}" mass="${wheel_mass}" mu="$(arg right_wheel_mu)" kp="$(arg wheel_kp)" width="$(arg wheel_width)"/>
+    <xacro:proximity_sensor tf_prefix="${tf_prefix}" group="proximity" range_max="$(arg proximity_max_range)" resolution="$(arg proximity_resolution)" fov="$(arg proximity_fov)" name="center" xyz="0.08 0 0.035" rpy="0 0 0"/>
+    <xacro:proximity_sensor tf_prefix="${tf_prefix}" group="proximity" range_max="$(arg proximity_max_range)" resolution="$(arg proximity_resolution)" fov="$(arg proximity_fov)" name="center_left" xyz="0.0756 0.0261 0.035" rpy="0 0 0.33161"/>
+    <xacro:proximity_sensor tf_prefix="${tf_prefix}" group="proximity" range_max="$(arg proximity_max_range)" resolution="$(arg proximity_resolution)" fov="$(arg proximity_fov)" name="center_right" xyz="0.0756 -0.0261 0.035" rpy="0 0 -0.33161"/>
+    <xacro:proximity_sensor tf_prefix="${tf_prefix}" group="proximity" range_max="$(arg proximity_max_range)" resolution="$(arg proximity_resolution)" fov="$(arg proximity_fov)" name="left" xyz="0.063 0.0493 0.035" rpy="0 0 0.66323"/>
+    <xacro:proximity_sensor tf_prefix="${tf_prefix}" group="proximity" range_max="$(arg proximity_max_range)" resolution="$(arg proximity_resolution)" fov="$(arg proximity_fov)" name="right" xyz="0.063 -0.0493 0.035" rpy="0 0 -0.66323"/>
+    <xacro:proximity_sensor tf_prefix="${tf_prefix}" group="proximity" range_max="$(arg proximity_max_range)" resolution="$(arg proximity_resolution)" fov="$(arg proximity_fov)" name="rear_left" xyz="-0.03 0.0305 0.035" rpy="0 0 3.14159"/>
+    <xacro:proximity_sensor tf_prefix="${tf_prefix}" group="proximity" range_max="$(arg proximity_max_range)" resolution="$(arg proximity_resolution)" fov="$(arg proximity_fov)" name="rear_right" xyz="-0.03 -0.0305 0.035" rpy="0 0 3.14159"/>
+    <xacro:proximity_sensor tf_prefix="${tf_prefix}" group="ground" range_max="0.03" name="left" xyz="0.07157 0.01155 0.0009" rpy="0 1.5708 0.24311"/>
+    <xacro:proximity_sensor tf_prefix="${tf_prefix}" group="ground" range_max="0.03" name="right" xyz="0.07157 -0.01155 0.0009" rpy="0 1.5708 -0.24311"/>
+    <link name="${tf_prefix}laser_link"/>
+    <joint name="${tf_prefix}base_laser_joint" type="fixed">
+      <parent link="${tf_prefix}base_link"/>
+      <child link="${tf_prefix}laser_link"/>
       <origin xyz="0 0 0.035"/>
     </joint>
-    <xacro:imu ns="$(arg name)"/>
+    <xacro:imu tf_prefix="${tf_prefix}"/>
     <!-- see https://github.com/ros-simulation/gazebo_ros_pkgs/blob/kinetic-devel/gazebo_plugins/src/gazebo_ros_diff_drive.cpp -->
     <gazebo>
@@ -88,8 +95,8 @@
         <odometrySource>encoder</odometrySource>
         <alwaysOn>true</alwaysOn>
-        <publishOdomTF>false</publishOdomTF>
+        <publishOdomTF>true</publishOdomTF>
         <updateRate>$(arg odom_max_rate)</updateRate>
-        <leftJoint>left_wheel_joint</leftJoint>
-        <rightJoint>right_wheel_joint</rightJoint>
+        <leftJoint>${tf_prefix}left_wheel_joint</leftJoint>
+        <rightJoint>${tf_prefix}right_wheel_joint</rightJoint>
         <wheelSeparation>${wheel_axis + 0 * r_wheel_width}</wheelSeparation>
         <wheelDiameter>${2 * wheel_radius}</wheelDiameter>
@@ -98,9 +105,9 @@
         <commandTopic>cmd_vel</commandTopic>
         <odometryTopic>odom</odometryTopic>
-        <odometryFrame>odom</odometryFrame>
+        <odometryFrame>${tf_prefix}odom</odometryFrame>
         <publishWheelJointState>true</publishWheelJointState>
         <publishWheelTF>false</publishWheelTF>
         <publishTf>true</publishTf>
-        <robotBaseFrame>base_link</robotBaseFrame>
+        <robotBaseFrame>${tf_prefix}base_link</robotBaseFrame>
       </plugin>
     </gazebo>
@@ -112,5 +119,5 @@
         <plugin name="ground_truth" filename="libgazebo_ros_p3d.so">
           <frameName>$(arg ground_truth_frame_id)</frameName>
-          <bodyName>base_link</bodyName>
+          <bodyName>${tf_prefix}base_link</bodyName>
           <topicName>ground_truth/odom</topicName>
           <updateRate>$(arg ground_truth_update_rate)</updateRate>

File: thymio_description/urdf/imu.urdf.xacro (robot description, xacro)
@@ -1,6 +1,6 @@
 <?xml version="1.0"?>
 <robot xmlns:xacro="http://playerstage.sourceforge.net/gazebo/xmlschema/#xacro">
-  <xacro:macro name="imu" params="ns">
-    <gazebo reference="base_link">
+  <xacro:macro name="imu" params="tf_prefix:=''">
+    <gazebo reference="${tf_prefix}base_link">
       <gravity>true</gravity>
       <sensor name="imu_sensor" type="imu">
@@ -11,10 +11,10 @@
         <plugin filename="libgazebo_ros_imu_sensor.so" name="imu_plugin">
           <topicName>imu</topicName>
-          <bodyName>base_link</bodyName>
+          <bodyName>${tf_prefix}base_link</bodyName>
           <updateRateHZ>16</updateRateHZ>
           <gaussianNoise>0.2646</gaussianNoise>
           <xyzOffset>0 0 0</xyzOffset>
           <rpyOffset>0 0 0</rpyOffset>
-          <frameName>${ns}base_link</frameName>
+          <frameName>${tf_prefix}base_link</frameName>
         </plugin>
         <pose>0 0 0 0 0 0</pose>

File: thymio_description/urdf/proximity_sensor.urdf.xacro (robot description, xacro)
@@ -1,12 +1,12 @@
 <?xml version="1.0"?>
 <robot xmlns:xacro="http://playerstage.sourceforge.net/gazebo/xmlschema/#xacro">
-  <xacro:macro name="proximity_sensor" params="group name xyz rpy update_rate:=10 range_min:=0.01 range_max:=0.12 resolution:=0.005 fov:=0.3">
-    <link name="${group}_${name}_link"/>
-    <joint name="${group}_${name}_joint" type="fixed">
+  <xacro:macro name="proximity_sensor" params="group name xyz rpy tf_prefix:='' update_rate:=10 range_min:=0.01 range_max:=0.12 resolution:=0.005 fov:=0.3">
+    <link name="${tf_prefix}${group}_${name}_link"/>
+    <joint name="${tf_prefix}${group}_${name}_joint" type="fixed">
       <origin xyz="${xyz}" rpy="${rpy}"/>
-      <parent link="base_link"/>
-      <child link="${group}_${name}_link"/>
+      <parent link="${tf_prefix}base_link"/>
+      <child link="${tf_prefix}${group}_${name}_link"/>
     </joint>
-    <gazebo reference="${group}_${name}_link">
+    <gazebo reference="${tf_prefix}${group}_${name}_link">
       <sensor name="${group}_${name}_sensor" type="ray">
         <visualize>true</visualize>
@@ -23,5 +23,5 @@
           <alwaysOn>true</alwaysOn>
           <updateRate>0</updateRate>
-          <frameName>${group}_${name}_link</frameName>
+          <frameName>${tf_prefix}${group}_${name}_link</frameName>
           <topicName>${group}/${name}</topicName>
           <radiation>infrared</radiation>

File: thymio_description/urdf/wheel.urdf.xacro (robot description, xacro)
@@ -1,6 +1,6 @@
 <?xml version="1.0"?>
 <robot xmlns:xacro="http://playerstage.sourceforge.net/gazebo/xmlschema/#xacro">
-  <xacro:macro name="wheel" params="name position mass:=0.024 mu:=100 radius:=0.022 width=0.015 max_speed=7.757 kp=10000">
-    <link name="${name}_wheel_link">
+  <xacro:macro name="wheel" params="name position tf_prefix:='' mass:=0.024 mu:=100 radius:=0.022 width=0.015 max_speed=7.757 kp=10000">
+    <link name="${tf_prefix}${name}_wheel_link">
       <inertial>
         <mass value="${mass}"/>
@@ -21,7 +21,7 @@
       </visual>
     </link>
-    <joint name="${name}_wheel_joint" type="continuous">
-      <parent link="base_link"/>
-      <child link="${name}_wheel_link"/>
+    <joint name="${tf_prefix}${name}_wheel_joint" type="continuous">
+      <parent link="${tf_prefix}base_link"/>
+      <child link="${tf_prefix}${name}_wheel_link"/>
       <axis xyz="0 1 0"/>
       <origin xyz="0 ${position} ${radius}"/>
@@ -29,5 +29,5 @@
       <!-- <dynamics damping="0.1" friction="0.1"/> -->
     </joint>
-    <gazebo reference="${name}_wheel_link">
+    <gazebo reference="${tf_prefix}${name}_wheel_link">
       <mu1>${mu}</mu1>
       <mu2>${mu / 2.0}</mu2>
